File: eurorack_to_breadboard_psu.kicad_sch (KiCad schematic)
At the start: 15 parts, among them J1 Conn_02x04_Odd_Even, J2 Conn_02x04_Odd_Even, J3 Conn_02x05_Odd_Even

Commit message: Fix page labels and add schematic pdf
Other:
- company: (none) -> RobotDialogs
- title: (none) -> Eurorack Breadboard PSU
Changed lines of the file:
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@@
 (kicad_sch (version 20211123) (generator eeschema)
   (paper "A4")
+  (title_block
+    (title "Eurorack Breadboard PSU")
+    (date "2022-01-22")
+    (rev "1")
+    (company "RobotDialogs")
+  )
   (junction (at 173.355 48.895) (diameter 0) (color 0 0 0 0)
   )
